Commit message: - Delete rgbd decleration from the main URDF file -Tailor the rgbd specs -Create a urdf file with required rgbd paramaters

File: schunk_robot/urdf/schunk_arm_with_rgbd.xacro (robot description, xacro)
@@ -2,4 +2,5 @@
 <robot name="schunk" xmlns:xacro="http://ros.org/wiki/xacro">
 <xacro:property name="M_PI" value="3.1415926535897931" />
+ <xacro:property name="deg_to_rad" value="0.01745329251994329577"/>
 <!--================================================================Gazebo References=============================================================================-->
 <gazebo reference="base_link">
@@ -284,4 +285,11 @@
     <dynamics damping="0.0" friction="0.0"/>
 </joint>
+<!--==================================== Sensor section======================================================== -->
+<xacro:include filename="$(find schunk_robot)/urdf/sensors/xtion_pro_live.urdf.xacro"/>
+<xacro:xtion_pro_live name="rgbd_camera" parent="base">
+    <!-- <origin xyz="0.5 0.0 0.8" rpy="0 ${75.0 * deg_to_rad} 0"/> -->
+    <origin xyz="0.5 0.0 0.8" rpy="0 0 ${-180.0 * deg_to_rad}"/>
+    <origin xyz="0 0 0" rpy="${-90.0 * deg_to_rad} 0 ${-90.0 * deg_to_rad}"/>
+  </xacro:xtion_pro_live>
 <!-- =================================== Transmissions for the joints ========================================== -->
 <!-- It seems that the Schunks joints are effort based, but we will use position based joints for now -->

File: schunk_robot/urdf/sensors/xtion_pro_live.gazebo.xacro (robot description, xacro)
@@ -6,11 +6,11 @@
       <sensor type="depth" name="${name}_frame_sensor">
         <always_on>true</always_on>
-        <update_rate>6.0</update_rate>
+        <update_rate>1.0</update_rate>
         <camera>
           <horizontal_fov>${58.0 * deg_to_rad}</horizontal_fov>
           <image>
             <format>R8G8B8</format>
-            <width>800</width>
-            <height>600</height>
+            <width>400</width>
+            <height>400</height>
           </image>
           <clip>
@@ -21,5 +21,5 @@
         <plugin name="${name}_frame_controller" filename="libgazebo_ros_openni_kinect.so">
           <alwaysOn>true</alwaysOn>
-          <updateRate>6.0</updateRate>
+          <updateRate>1.0</updateRate>
           <cameraName>${name}</cameraName>
           <imageTopicName>ir/image_raw</imageTopicName>
@@ -43,10 +43,10 @@
       <sensor type="depth" name="${name}_frame_sensor">
         <always_on>true</always_on>
-        <update_rate>6.0</update_rate>
+        <update_rate>1.0/update_rate>
         <camera>
           <horizontal_fov>${58.0 * deg_to_rad}</horizontal_fov>
           <image>
             <format>R8G8B8</format>
-            <width>800</width>
+            <width>400</width>
             <height>600</height>
           </image>
@@ -58,5 +58,5 @@
         <plugin name="${name}_frame_controller" filename="libgazebo_ros_openni_kinect.so">
           <alwaysOn>true</alwaysOn>
-          <updateRate>6.0</updateRate>
+          <updateRate>1.0</updateRate>
           <cameraName>${name}</cameraName>
           <imageTopicName>rgb/image_raw</imageTopicName>
