Commit message: schunk arm urdf completed - test urdf file deleted

File: schunk_robot/urdf/schunk_arm.xacro (robot description, xacro)
@@ -18,9 +18,9 @@
     <material value="Gazebo/Green"/>
 </gazebo>
-<!-- <gazebo reference="joint3">
+<gazebo reference="link3">
     <gravity>true</gravity>
     <self_collide>false</self_collide>
     <material value="Gazebo/Blue"/>
-</gazebo> -->
+</gazebo>
 <!-- <gazebo reference="joint4">
     <gravity>true</gravity>
@@ -56,6 +56,6 @@
             <mesh filename="package://schunk_robot/meshes/robot_base_v3.STL"/>
         </geometry>
-        <material name="blue">
-            <color rgba="0 0 1 1"/>
+        <material name="red">
+            <color rgba="1 0 0 1"/>
         </material>
     </visual>
@@ -87,6 +87,6 @@
             <mesh filename="package://schunk_robot/meshes/joint1_v3.STL"/>
         </geometry>
-        <material name="red">
-            <color rgba="1 0 0 1"/>
+        <material name="green">
+            <color rgba="0 1 0 1"/>
         </material>
     </visual>
@@ -115,5 +115,5 @@
 </joint>
 <!--================================================================Link 2====================================================================================-->
-<!-- <link name="link2">
+<link name="link2">
     <visual>
         <origin rpy="0 0 0" xyz="0 0.005 0"/>
@@ -121,5 +121,7 @@
             <mesh filename="package://schunk_robot/meshes/joint2_v3.STL"/>
         </geometry>
-        <material name="Neobotix/Green"/>
+        <material name="blue">
+            <color rgba="0 0 1 1"/>
+        </material>
     </visual>
     <collision>
@@ -129,7 +131,7 @@
         </geometry>
     </collision>
-    <inertial> -->
-        <!--mass value="2"/-->
-        <!-- <mass value="2.5"/>
+    <inertial>
+        <!--mass value="2"/-->
+         <mass value="2.5"/>
         <origin xyz="0 -0.1925 0" rpy="0 0 0"/>
         <inertia ixx="0.030278"	 ixy="-0.007138" ixz="0.000435"
@@ -137,6 +139,6 @@
                  izx="0.000435"	 izy=" 0.000859" izz="0.030724"/>
     </inertial>
-</link> -->
-<!-- <joint name="joint2" type="revolute">
+</link>
+<joint name="joint2" type="revolute">
     <axis xyz="0 0 1"/>
     <limit effort="1000.0" lower="-2.0071" upper="2.0071" velocity="0.5"/>
@@ -145,4 +147,140 @@
     <origin xyz="0 0 0.165" rpy="-1.57079 0 0"/>
     <dynamics damping="0.0" friction="0.0"/>
-</joint> -->
+</joint>
+<!--================================================================Link 3====================================================================================-->
+<link name="link3">
+    <visual>
+        <origin xyz="0 0 0" rpy="0 0 0"/>
+        <geometry>
+            <mesh filename="package://schunk_robot/meshes/joint3_v3.STL"/>
+        </geometry>
+        <material name="red">
+            <color rgba="1 0 0 1"/>
+        </material>
+    </visual>
+    <collision>
+        <origin xyz="0 0 0" rpy="0 0 0"/>
+        <geometry>
+            <mesh filename="package://schunk_robot/meshes/joint3_v3.STL"/>
+        </geometry>
+    </collision>
+    <inertial>
+        <!--mass value="2"/-->
+        <mass value="2.5"/>
+        <origin xyz="0 0 0" rpy="0 0 0"/>
+        <inertia ixx="0.002573" ixy="0.000000" ixz="0.000000"
+                 iyx="0.000000" iyy="0.003196" iyz="0.000000"
+                 izx="0.000000" izy="0.000000" izz="0.002484"/>
+    </inertial>
+</link>
+<joint name="joint3" type="revolute">
+    <axis xyz="0 0 1"/>
+    <limit effort="1000.0" lower="-1.9199" upper="1.9199" velocity="0.5"/>
+    <parent link="link2"/>
+    <child link="link3"/>
+    <origin xyz="0 -0.385 0" rpy="0 0 0"/>
+    <dynamics damping="0.0" friction="0.0"/>
+</joint>
+<!--================================================================Link 4====================================================================================-->
+<link name="link4">
+    <visual>
+        <origin xyz="0 0 0.4445" rpy="0 0 0" />
+        <geometry>
+            <mesh filename="package://schunk_robot/meshes/joint4_v3.STL"/>
+        </geometry>
+        <material name="green">
+            <color rgba="0 1 0 1"/>
+        </material>
+    </visual>
+    <collision>
+        <origin xyz="0 0 0.4445" rpy="0 0 0"/>
+        <geometry>
+            <mesh filename="package://schunk_robot/meshes/joint4_v3.STL"/>
+        </geometry>
+    </collision>
+    <inertial>
+        <!--mass value="2"/-->
+        <mass value="1.7"/>
+        <origin xyz="0 0 0.2225" rpy="1.57079 1.57079 0"/>
+        <inertia ixx="0.003830"  ixy="0.001706"  ixz="-0.003042"
+                 iyx="0.001706"  iyy="0.010112"  iyz="-0.000765"
+                 izx="-0.003042" izy="-0.000765" izz="0.009108"/>
+    </inertial>
+</link>
+<joint name="joint4" type="revolute">
+    <axis xyz="0 0 1"/>
+    <limit effort="1000.0" lower="-3.4907" upper="3.4907" velocity="0.5"/>
+    <parent link="link3"/>
+    <child link="link4"/>
+    <origin xyz="0 0 0" rpy="1.57079 0 0"/>
+    <dynamics damping="0.0" friction="0.0"/>
+</joint>
+<!--================================================================Link 5====================================================================================-->
+<link name="link5">
+    <visual>
+        <origin xyz="0 0 0" rpy="1.57079 0 3.14159"/>
+        <geometry>
+            <mesh filename="package://schunk_robot/meshes/joint5_v3.STL"/>
+        </geometry>
+        <material name="blue">
+            <color rgba="0 0 1 1"/>
+        </material>
+    </visual>
+    <collision>
+        <origin xyz="0 0 0" rpy="1.57079 0 3.14159"/>
+        <geometry>
+            <mesh filename="package://schunk_robot/meshes/joint5_v3.STL"/>
+        </geometry>
+    </collision>
+    <inertial>
+        <!--mass value="2"/-->
+        <mass value="1.6"/>
+        <origin xyz="0 0 0" rpy="0 0 0"/>
+        <inertia ixx="0.001222" ixy="0.000061" ixz="0.000141"
+                 iyx="0.000061" iyy="0.001793" iyz="0.000048"
+                 izx="0.000141" izy="0.000048" izz="0.001435"/>
+    </inertial>
+</link>
+<joint name="joint5" type="revolute">
+    <axis xyz="0 0 1"/>
+    <limit effort="1000.0" lower="-1.8675" upper="1.8675" velocity="0.5"/>
+    <parent link="link4"/>
+    <child link="link5"/>
+    <origin  xyz="0 0 0.445" rpy="-1.57079 0 0"/>
+    <dynamics damping="0.0" friction="0.0"/>
+</joint>
+<!--================================================================Link 6====================================================================================-->
+<link name="link6">
+    <visual>
+        <origin rpy="0 0 0" xyz="0 0 0"/>
+        <geometry>
+            <mesh filename="package://schunk_robot/meshes/joint6_v3.STL"/>
+        </geometry>
+        <material name="yellow">
+            <color rgba="1 1 0 1"/>
+        </material>
+    </visual>
+    <collision>
+        <origin rpy="0 0 0" xyz="0 0 0"/>
+        <geometry>
+              <mesh filename="package://schunk_robot/meshes/joint6_v3.STL"/>
+        </geometry>
+    </collision>
+    <inertial>
+        <!--mass value="2"/-->
+        <mass value="1.6"/>
+        <origin xyz="0 0 -0.06" rpy="0 0 0"/>
+        <inertia ixx="0.000654" ixy="0.000000" ixz="0.000000"
+                 iyx="0.000000" iyy="0.000954" iyz="0.000000"
+                 izx="0.000000" izy="0.000000" izz="0.000929"/>
+    </inertial>
+</link>
+<joint name="joint6" type="revolute">
+    <origin xyz="0 -0.2 0" rpy="1.57079 0 0" />
+    <axis xyz="0 0 1"/>
+    <limit effort="1000.0" lower="-3.4907" upper="3.4907" velocity="0.5"/>
+    <parent link="link5"/>
+    <child link="link6"/>
+    <dynamics damping="0.0" friction="0.0"/>
+</joint>
 </robot>

Commit message: -schunk xacro updated with gazebo color tags -launch file created to spawn the arm in gazebo(no controls)

File: schunk_robot/urdf/schunk_arm.xacro (robot description, xacro)
@@ -3,41 +3,41 @@
 <xacro:property name="M_PI" value="3.1415926535897931" />
 <!--================================================================Gazebo References=============================================================================-->
-<gazebo reference="robot_base">
+<gazebo reference="base_link">
+    <gravity>true</gravity>
+    <self_collide>false</self_collide>
+    <material value="Gazebo/Red"/>
+</gazebo>
+<gazebo reference="link1">
+    <gravity>true</gravity>
+    <self_collide>false</self_collide>
+    <material value="Gazebo/Green"/>
+</gazebo>
+<gazebo reference="link2">
     <gravity>true</gravity>
     <self_collide>false</self_collide>
     <material value="Gazebo/Blue"/>
 </gazebo>
-<gazebo reference="link1">
+<gazebo reference="link3">
     <gravity>true</gravity>
     <self_collide>false</self_collide>
     <material value="Gazebo/Red"/>
 </gazebo>
-<gazebo reference="link2">
+<gazebo reference="link4">
     <gravity>true</gravity>
     <self_collide>false</self_collide>
     <material value="Gazebo/Green"/>
 </gazebo>
-<gazebo reference="link3">
+<gazebo reference="link5">
     <gravity>true</gravity>
     <self_collide>false</self_collide>
     <material value="Gazebo/Blue"/>
 </gazebo>
-<!-- <gazebo reference="joint4">
-    <gravity>true</gravity>
-    <self_collide>false</self_collide>
-    <material value="Gazebo/Red"/>
-</gazebo> -->
-<!-- <gazebo reference="joint5">
-    <gravity>true</gravity>
-    <self_collide>false</self_collide>
-    <material value="Gazebo/Green"/>
-</gazebo> -->
-<!-- <gazebo reference="joint6">
-    <gravity>true</gravity>
-    <self_collide>false</self_collide>
-    <material value="Gazebo/Blue"/>
-    minDepth for magnetic gripper
+<gazebo reference="link6">
+    <gravity>true</gravity>
+    <self_collide>false</self_collide>
+    <material value="Gazebo/Yellow"/>
+    <!-- minDepth for magnetic gripper -->
     <minDepth>0.02</minDepth>
-</gazebo> -->
+</gazebo>
 <!-- <gazebo>
   <plugin name="gazebo_ros_control" filename="libgazebo_ros_control.so">

Commit message: -Add transmission tags to the URDF for gazebo control

File: schunk_robot/urdf/schunk_arm.xacro (robot description, xacro)
@@ -40,9 +40,9 @@
     <minDepth>0.02</minDepth>
 </gazebo>
-<!-- <gazebo>
+<gazebo>
   <plugin name="gazebo_ros_control" filename="libgazebo_ros_control.so">
     <robotNamespace>/schunk</robotNamespace>
   </plugin>
-</gazebo> -->
+</gazebo>
 <!--===================================================+==========Schunk Arm====================================================================================-->
 <!--===================================================+========= Schunk arm connection to world ====================================================================================-->
@@ -286,3 +286,65 @@
 <!--==================================== Sensor section======================================================== -->
 <xacro:include filename="$(find schunk_robot)/urdf/sensors/xtion_pro_live.urdf.xacro"/>
+<!-- =================================== Transmissions for the joints ========================================== -->
+<!-- It seems that the Schunks joints are effort based, but we will use position based joints for now -->
+<transmission name="joint1_trans">
+    <type>transmission_interface/SimpleTransmission</type>
+    <joint name="joint1">
+        <hardwareInterface>hardware_interface/PositionJointInterface</hardwareInterface>
+    </joint>
+    <actuator name="joint1_motor">
+        <hardwareInterface>hardware_interface/PositionJointInterface</hardwareInterface>
+        <mechanicalReduction>1</mechanicalReduction>
+    </actuator>
+</transmission>
+<transmission name="joint2_trans">
+    <type>transmission_interface/SimpleTransmission</type>
+    <joint name="joint2">
+        <hardwareInterface>hardware_interface/PositionJointInterface</hardwareInterface>
+    </joint>
+    <actuator name="joint2_motor">
+        <hardwareInterface>hardware_interface/PositionJointInterface</hardwareInterface>
+        <mechanicalReduction>1</mechanicalReduction>
+    </actuator>
+</transmission>
+<transmission name="joint3_trans">
+    <type>transmission_interface/SimpleTransmission</type>
+    <joint name="joint3">
+        <hardwareInterface>hardware_interface/PositionJointInterface</hardwareInterface>
+    </joint>
+    <actuator name="joint3_motor">
+        <hardwareInterface>hardware_interface/PositionJointInterface</hardwareInterface>
+        <mechanicalReduction>1</mechanicalReduction>
+    </actuator>
+</transmission>
+<transmission name="joint4_trans">
+    <type>transmission_interface/SimpleTransmission</type>
+    <joint name="joint4">
+        <hardwareInterface>hardware_interface/PositionJointInterface</hardwareInterface>
+    </joint>
+    <actuator name="joint4_motor">
+        <hardwareInterface>hardware_interface/PositionJointInterface</hardwareInterface>
+        <mechanicalReduction>1</mechanicalReduction>
+    </actuator>
+</transmission>
+<transmission name="joint5_trans">
+    <type>transmission_interface/SimpleTransmission</type>
+    <joint name="joint5">
+        <hardwareInterface>hardware_interface/PositionJointInterface</hardwareInterface>
+    </joint>
+    <actuator name="joint5_motor">
+        <hardwareInterface>hardware_interface/PositionJointInterface</hardwareInterface>
+        <mechanicalReduction>1</mechanicalReduction>
+    </actuator>
+</transmission>
+<transmission name="joint6_trans">
+    <type>transmission_interface/SimpleTransmission</type>
+    <joint name="joint6">
+        <hardwareInterface>hardware_interface/PositionJointInterface</hardwareInterface>
+    </joint>
+    <actuator name="joint6_motor">
+        <hardwareInterface>hardware_interface/PositionJointInterface</hardwareInterface>
+        <mechanicalReduction>1</mechanicalReduction>
+    </actuator>
+</transmission>
 </robot>

Commit message: - Add package for training data generation -Add visual scene Gazebo plugin to schunk xacro (gazebo section)

File: schunk_robot/urdf/schunk_arm.xacro (robot description, xacro)
@@ -59,4 +59,7 @@
             <color rgba="1 0 0 1"/>
         </material>
+        <!-- Gazebo visual plugin for changing the background of the scene -->
+        <plugin name="visual_scene_edit" filename="libvisual_scene_edit.so">
+        </plugin>
     </visual>
     <collision>

File: schunk_robot/urdf/schunk_arm_with_rgbd.xacro (robot description, xacro)
@@ -8,4 +8,8 @@
     <self_collide>false</self_collide>
     <material value="Gazebo/Red"/>
+    <!-- Gazebo visual plugin for changing the background of the scene -->
+    <visual>
+        <plugin name="visual_scene_edit" filename="libvisual_scene_edit.so"/>
+    </visual>
 </gazebo>
 <gazebo reference="link1">
